File: ESP32-Telemetry/ESP32-Telemetry.kicad_pcb (KiCad board)
At the start: 2 copper layers, 30 parts, among them J1 USB_B_Micro, J2 CJMCU-811, J3 DS18B20, J4 LEDs, Q1 2N7002, SW1 Reset, SW2 Prog, U1 NCP1117-3.3_SOT223, U2 FT230XS, U3 ESP32-WROOM-32D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

Commit message: Starting on PCB layout...
Parts:
- moved J1 70.7 mm to (106.8, 87.7), turned to 270 degrees
- moved C1 61.0 mm to (115.2, 80.2), turned to 90 degrees
- moved J3 57.7 mm to (203.8, 119.3)
- moved J4 55.6 mm to (204.1, 106.9)
- moved J2 55.3 mm to (203.8, 80.6)
- moved C2 53.5 mm to (118.1, 80.1), turned to 90 degrees
- moved U1 47.6 mm to (120.1, 70.8), turned to 270 degrees
- moved R1 46.9 mm to (124.8, 80.2), turned to 270 degrees
- moved SW1 42.1 mm to (109.9, 101.6), turned to 180 degrees
- moved SW2 41.0 mm to (123.3, 101.7), turned to 180 degrees
- moved U2 40.1 mm to (124.5, 87.5), turned to 90 degrees
- moved R3 40.0 mm to (121.2, 92.8), turned to 180 degrees
- moved FB2 38.2 mm to (116.1, 85.1)
- moved U5 33.3 mm to (194.7, 71.2)
- moved C5 31.8 mm to (164.6, 88.0)
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
Commit message: First shot at layout...
Parts:
- moved J2 86.6 mm to (117.8, 71.5), turned to 90 degrees
- moved J4 70.1 mm to (143.5, 71.5), turned to 90 degrees
- moved J3 66.3 mm to (157.5, 71.8), turned to 90 degrees
- moved R6 42.7 mm to (128.5, 86.8), turned to 270 degrees
- moved R4 41.7 mm to (129.8, 78.4), turned to 270 degrees
- moved R5 38.7 mm to (128.0, 92.7)
- moved U5 30.4 mm to (165.2, 78.8)
- moved R2 25.9 mm to (158.5, 102.5)
- moved Q1 23.8 mm to (158.5, 81.5), turned to 270 degrees
- moved R10 23.2 mm to (158.5, 76.7)
- moved R7 17.3 mm to (158.5, 86.3)
- moved R9 13.9 mm to (158.5, 90.4), turned to 180 degrees
- moved U1 12.5 mm to (109.7, 77.7), turned to 90 degrees
- moved C5 12.1 mm to (158.5, 98.4), turned to 180 degrees
- moved R11 11.3 mm to (165.1, 89.4)
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
Commit message: WIP layout. Bit of a 🚮🔥 at the moment.
Parts:
- moved R10 13.7 mm to (144.8, 75.7)
- moved R2 8.52 mm to (158.5, 94.0), turned to 180 degrees
- moved R11 3.21 mm to (166.1, 86.4)
- moved R8 2.88 mm to (158.5, 97.3), turned to 180 degrees
- moved C5 2.14 mm to (158.5, 100.6)
- moved C4 1.65 mm to (117.6, 92.8), turned to 90 degrees
- moved R5 0.92 mm to (128.5, 91.9), turned to 270 degrees
- turned FB2 to 180 degrees
- turned Q1 to 90 degrees
- turned R1 to 90 degrees
- turned R3 to 270 degrees
- turned R6 to 90 degrees
Connections:
- J1 pad 4: (no net) -> Net-(J1-Pad4)
- J2 pad 6: (no net) -> Net-(J2-Pad6)
- J2 pad 7: (no net) -> Net-(J2-Pad7)
- J2 pad 8: (no net) -> Net-(J2-Pad8)
- Q1 pad 2: (no net) -> GND
- U2 pad 14: (no net) -> Net-(U2-Pad14)
- U2 pad 15: (no net) -> Net-(U2-Pad15)
- U2 pad 16: (no net) -> Net-(U2-Pad16)
- U2 pad 6: (no net) -> Net-(U2-Pad6)
- U2 pad 7: (no net) -> Net-(U2-Pad7)
- U3 pad 12: (no net) -> Net-(U3-Pad12)
- U3 pad 13: (no net) -> Net-(U3-Pad13)
- U3 pad 14: (no net) -> Net-(U3-Pad14)
- U3 pad 16: (no net) -> Net-(U3-Pad16)
- U3 pad 17: (no net) -> Net-(U3-Pad17)
- U3 pad 18: (no net) -> Net-(U3-Pad18)
- U3 pad 19: (no net) -> Net-(U3-Pad19)
- U3 pad 20: (no net) -> Net-(U3-Pad20)
- U3 pad 21: (no net) -> Net-(U3-Pad21)
- U3 pad 22: (no net) -> Net-(U3-Pad22)
- U3 pad 23: (no net) -> Net-(U3-Pad23)
- U3 pad 24: (no net) -> Net-(U3-Pad24)
- U3 pad 26: (no net) -> Net-(U3-Pad26)
- U3 pad 27: (no net) -> Net-(U3-Pad27)
- U3 pad 28: (no net) -> Net-(U3-Pad28)
- U3 pad 29: (no net) -> Net-(U3-Pad29)
- U3 pad 30: (no net) -> Net-(U3-Pad30)
- U3 pad 31: (no net) -> Net-(U3-Pad31)
- U3 pad 4: (no net) -> Net-(U3-Pad4)
- U3 pad 5: (no net) -> Net-(U3-Pad5)
- U3 pad 6: (no net) -> Net-(U3-Pad6)
- U3 pad 7: (no net) -> Net-(U3-Pad7)
- U3 pad 8: (no net) -> Net-(U3-Pad8)
- U3 pad 9: (no net) -> Net-(U3-Pad9)
- U5 pad 3: (no net) -> Net-(U5-Pad3)
Routing:
- net +3V3: track 0.00 -> 161.0 mm
- net /DS18B20-Data: track 0.00 -> 45.1 mm
- net GND: track 0.00 -> 42.4 mm, vias 0 -> 26
- net +5V: track 0.00 -> 25.9 mm
- net Net-(U2-Pad1): track 0.00 -> 25.0 mm
- net Net-(J4-Pad2): track 0.00 -> 19.4 mm
- net Net-(R1-Pad1): track 0.00 -> 19.3 mm
- net Net-(J1-Pad2): track 0.00 -> 18.3 mm
- net Net-(J1-Pad3): track 0.00 -> 17.3 mm
- net Net-(C4-Pad1): track 0.00 -> 15.6 mm
- net Net-(R4-Pad2): track 0.00 -> 13.7 mm
- net Net-(Q1-Pad1): track 0.00 -> 11.7 mm
- net /LEDs-Data: track 0.00 -> 10.5 mm
- net Net-(R11-Pad2): track 0.00 -> 10.5 mm
- net Net-(FB2-Pad2): track 0.00 -> 7.46 mm
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- added copper zone on F.Cu, net +3V3
- added copper zone on B.Cu, net GND

Commit message: WIP routing
Parts:
- moved J2 18.1 mm to (135.9, 71.8), turned to 270 degrees
- moved R9 11.4 mm to (157.5, 79.0), turned to 270 degrees
- moved R11 10.3 mm to (164.5, 76.2)
- moved Q1 8.96 mm to (151.8, 75.6), turned to 180 degrees
- moved R8 5.37 mm to (161.3, 92.7), turned to 90 degrees
- moved C1 5.31 mm to (121.3, 78.5)
- moved C3 5.00 mm to (118.5, 76.0)
- moved R6 4.80 mm to (129.5, 91.4), turned to 0 degrees
- moved C5 3.57 mm to (157.5, 97.2), turned to 90 degrees
- moved R5 3.45 mm to (129.5, 95.2), turned to 0 degrees
- moved C2 3.43 mm to (116.0, 78.5)
- moved R4 2.88 mm to (129.5, 81.3), turned to 0 degrees
- moved U5 2.61 mm to (164.6, 81.3)
- moved R1 2.11 mm to (124.5, 79.4), turned to 180 degrees
- moved U4 2.08 mm to (165.1, 94.6), turned to 270 degrees
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Routing:
- net +3V3: track 161.0 -> 132.9 mm
- net Net-(U2-Pad1): track 25.0 -> 0.00 mm
- net Net-(R1-Pad1): track 19.3 -> 4.63 mm
- net Net-(J4-Pad2): track 19.4 -> 9.30 mm
- net /DS18B20-Data: track 45.1 -> 52.3 mm
- net Net-(Q1-Pad1): track 11.7 -> 5.31 mm
- net Net-(R11-Pad2): track 10.5 -> 5.90 mm
- net SDA: track 0.00 -> 3.94 mm
- net +5V: track 25.9 -> 22.5 mm
- net SCL: track 7.20 -> 3.94 mm
- net /LEDs-Data: track 10.5 -> 13.7 mm
- net Net-(R1-Pad2): track 7.24 -> 5.12 mm
- net Net-(R4-Pad2): track 13.7 -> 11.9 mm
- net GND: track 42.4 -> 41.0 mm, vias 26 -> 28
- net Net-(R2-Pad2): track 6.90 -> 7.45 mm
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
Commit message: As submitted 2020-02-15
Parts:
- moved R3 0.25 mm to (121.2, 93.0)
Routing:
- net SCL: track 3.94 -> 59.1 mm, vias 0 -> 3
- net SDA: track 3.94 -> 56.1 mm, vias 0 -> 2
- net /CCS811-Wake: track 0.00 -> 34.7 mm, vias 0 -> 1
- net Net-(R2-Pad2): track 7.45 -> 39.2 mm, vias 0 -> 2
- net +3V3: track 132.9 -> 158.1 mm
- net +5V: track 22.5 -> 46.5 mm, vias 0 -> 2
- net Net-(R4-Pad2): track 11.9 -> 32.8 mm, vias 0 -> 2
- net Net-(U2-Pad1): track 0.00 -> 18.4 mm, vias 0 -> 2
- net Net-(U2-Pad4): track 0.00 -> 15.6 mm, vias 0 -> 2
- net Net-(R1-Pad1): track 4.63 -> 14.0 mm, vias 0 -> 2
- net GND: track 41.0 -> 45.8 mm, vias 28 -> 29
Other:
- board outline added: 68 x 40 mm
